File: model/jtdd/jtdd.sch (KiCad schematic (older format))
At the start: 18 parts

Commit message: timing sim
Parts:
- removed U? (x3): 7400, symbol jt74xx:7400
- added U1, U9: 74HC04, symbol jt74xx:74HC04
- added U10, U2: 74LS112, symbol jt74xx:74LS112
- added U11, U13, U34, U6: 74LS00, symbol jt74xx:74LS00
- added U14, U15, U16, U17, U18, U19, U20, U21: 74HC86, symbol jt74xx:74HC86
- added U31, U33: 74LS273, symbol jt74xx:74LS273
- added U32: 74LS30, symbol jt74xx:74LS30
- added U7, U8: 74LS161, symbol jt74xx:74LS161
- gave numbers to parts that had none: 15
Connections:
- net labels added: DVPOS[0], DVPOS[1], DVPOS[2], DVPOS[3], DVPOS[4], DVPOS[5], DVPOS[6], DVPOS[7], HN[0], HN[1], HN[2], HN[3], HN[4], HN[5], HN[6], HN[7], HN[8], HPOS[0], HPOS[1], HPOS[2], HPOS[3], HPOS[4], HPOS[5], HPOS[6], HPOS[7], RSTn, VBLK, VN[0], VN[1], VN[2], VN[3], VN[4], VN[5], VN[6], VN[7], VPOS[0], VPOS[1], VPOS[2], VPOS[3], VPOS[4], VPOS[5], VPOS[6], VPOS[7], flipn, hc0, hc1, hover
- wire segments 111 -> 274

Commit message: Timing simulation. Colour mix done
Parts:
- added U?: 74HC04, symbol jt74xx:74HC04
- added U?: 74LS74, symbol jt74xx:74LS74
Connections:
- net HN[0]: now also U?.1
- net HN[8]: now also U10.1 (C), U2.1 (C)
- net tie1: now also U?.1 (~R), U?.4 (~S)
- net HCLK1: now reaches U12.3 (O1a)
- net HCLK1: now also U?.3 (C)
- net at U31.11 (Cp), U33.11 (Cp), U7.2 (CP)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: now also U8.2 (CP)
- new net E: U?.2, U?.2 (D)
- new net Q: U?.6 (~Q)
- no-connect marks 1 -> 2
Changed lines of the file:
@@
 	1950 6350 1950 7500
 Wire Wire Line
-	1950 7500 2500 7500
+	1950 7500 2100 7500
 Wire Wire Line
 	2500 6700 2400 6700
@@
 	-1   0    0    1
 $EndComp
-Connection ~ 3300 6100
-Connection ~ 3300 5900
-Connection ~ 2700 6000
 $Comp
 L jt74xx:74LS00 U13
@@
 Text Label 3700 4150 0    50   ~ 0
 hc1
+Wire Wire Line
+	2100 7500 2100 9050
+Wire Wire Line
+	2100 9050 2500 9050
+Connection ~ 2100 7500
+Wire Wire Line
+	2100 7500 2500 7500
+Text Label 2550 10500 0    50   ~ 0
+HN[8]
+Wire Wire Line
+	4900 1400 5900 1400
+Text Label 5250 1400 0    50   ~ 0
+HCLK1
+$Comp
+L jt74xx:74HC04 U?
+U 1 1 5E281C6A
+P 9000 1500
+F 0 "U?" V 8954 1680 50  0000 L CNN
+F 1 "74HC04" V 9045 1680 50  0000 L CNN
+F 2 "" H 9000 1500 50  0001 C CNN
+F 3 "http://www.nxp.com/documents/data_sheet/74HC_HCT04.pdf" H 9000 1500 50  0001 C CNN
+	1    9000 1500
+	1    0    0    -1
+$EndComp
+$Comp
+L jt74xx:74LS74 U?
+U 1 1 5E281E38
+P 10000 2200
+F 0 "U?" H 10000 2678 50  0000 C CNN
+F 1 "74LS74" H 10000 2587 50  0000 C CNN
+F 2 "" H 10000 2200 50  0001 C CNN
+F 3 "74xx/74hc_hct74.pdf" H 10000 2200 50  0001 C CNN
+	1    10000 2200
+	1    0    0    -1
+$EndComp
+Wire Wire Line
+	8700 1500 8450 1500
+Text Label 8450 1500 0    50   ~ 0
+HN[0]
+Wire Wire Line
+	9300 1500 9400 1500
+Text GLabel 9550 1500 2    50   Output ~ 0
+E
+Wire Wire Line
+	9400 1500 9400 2100
+Wire Wire Line
+	9400 2100 9700 2100
+Connection ~ 9400 1500
+Wire Wire Line
+	9400 1500 9550 1500
+Wire Wire Line
+	9700 2200 9400 2200
+Text Label 9400 2200 2    50   ~ 0
+HCLK1
+Text Label 10000 1900 2    50   ~ 0
+tie1
+Text Label 10000 2500 3    50   ~ 0
+tie1
+Wire Wire Line
+	10300 2300 10500 2300
+Text GLabel 10500 2300 2    50   Output ~ 0
+Q
+NoConn ~ 10300 2100
 $EndSCHEMATC

Commit message: MCU WIP
Parts:
- gave numbers to parts that had none: 2
Changed lines of the file:
@@
 HCLK1
 $Comp
-L jt74xx:74HC04 U?
+L jt74xx:74HC04 U35
 U 1 1 5E281C6A
 P 9000 1500
-F 0 "U?" V 8954 1680 50  0000 L CNN
+F 0 "U35" V 8954 1680 50  0000 L CNN
 F 1 "74HC04" V 9045 1680 50  0000 L CNN
 F 2 "" H 9000 1500 50  0001 C CNN
@@
 $EndComp
 $Comp
-L jt74xx:74LS74 U?
+L jt74xx:74LS74 U36
 U 1 1 5E281E38
 P 10000 2200
-F 0 "U?" H 10000 2678 50  0000 C CNN
+F 0 "U36" H 10000 2678 50  0000 C CNN
 F 1 "74LS74" H 10000 2587 50  0000 C CNN
 F 2 "" H 10000 2200 50  0001 C CNN
